File: power-switch-ch.sch (KiCad schematic (older format))
At the start: 8 parts, among them J1 Screw_Terminal_1x02, K1 RELAY, Q1 2N2222

Commit message: use official footprint libs
Parts:
- K1: footprint IHE:Relay -> Relay_THT:Relay_SPST_TE_PCN-1xxD3MHZ
- R1: value 10kΩ -> 240Ω
Changed lines of the file:
@@
 AR Path="/5BA1E15E/5BA1D969" Ref="R4"  Part="1"
 F 0 "R1" V 4430 3900 50  0000 C CNN
-F 1 "10kΩ" V 4350 3900 50  0000 C CNN
+F 1 "240Ω" V 4350 3900 50  0000 C CNN
 F 2 "Resistors_SMD:R_0805_HandSoldering" V 4280 3900 50  0001 C CNN
 F 3 "" H 4350 3900 50  0000 C CNN
@@
 AR Path="/5BA1E081/5BA1D972" Ref="#PWR07"  Part="1"
 AR Path="/5BA1E15E/5BA1D972" Ref="#PWR09"  Part="1"
-F 0 "#PWR05" H 4950 4000 50  0001 C CNN
+F 0 "#PWR03" H 4950 4000 50  0001 C CNN
 F 1 "GND" H 4950 4100 50  0000 C CNN
 F 2 "" H 4950 4250 50  0000 C CNN
@@
 F 0 "K1" H 5450 3150 60  0000 C CNN
 F 1 "RELAY" H 5450 3350 60  0000 C CNN
-F 2 "IHE:Relay" H 5450 3200 60  0001 C CNN
+F 2 "Relay_THT:Relay_SPST_TE_PCN-1xxD3MHZ" H 5450 3200 60  0001 C CNN
 F 3 "" H 5450 3200 60  0000 C CNN
 	1    5450 3200
@@
 AR Path="/5BA1E081/5BA1D994" Ref="#PWR08"  Part="1"
 AR Path="/5BA1E15E/5BA1D994" Ref="#PWR010"  Part="1"
-F 0 "#PWR06" H 4950 2650 50  0001 C CNN
+F 0 "#PWR04" H 4950 2650 50  0001 C CNN
 F 1 "+5V" H 4950 2940 50  0000 C CNN
 F 2 "" H 4950 2800 50  0000 C CNN
