File: power-switching-driver.kicad_pcb (KiCad board)
At the start: 2 copper layers, 48 x 48 mm, 21 parts, among them J1 Screw_Terminal_1x02, J2 Screw_Terminal_1x02, K1 RELAY, K2 RELAY, P1 CONN_02X02, Q1 2N2222, Q2 2N2222

Commit message: use updated footprint locally until pull request comes through
Parts:
- K2: footprint IHE:Relay -> IHE2:Relay
Routing:
- net Net-(J2-Pad2): track 11.9 -> 13.7 mm
- net Net-(J1-Pad2): track 11.9 -> 13.7 mm
Other:
- board text added: "Rev B"
Changed lines of the file:
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@@
-(kicad_pcb (version 4) (host pcbnew 4.0.4-stable)
+(kicad_pcb (version 20171130) (host pcbnew "(5.0.0-3-g5ebb6b6)")
   (general
-    (links 26)
-    (no_connects 0)
-    (area 124.274999 73.074999 172.425001 126.225001)
     (thickness 1.6)
-    (drawings 6)
-    (tracks 54)
+    (drawings 7)
+    (tracks 58)
     (zones 0)
     (modules 21)
@@
       (layerselection 0x00030_80000001)
       (usegerberextensions false)
+      (usegerberattributes false)
+      (usegerberadvancedattributes false)
+      (creategerberjobfile false)
       (excludeedgelayer true)
       (linewidth 0.100000)
@@
       (hpglpennumber 1)
       (hpglpenspeed 20)
-      (hpglpendiameter 15)
-      (hpglpenoverlay 2)
+      (hpglpendiameter 15.000000)
       (psnegative false)
       (psa4output false)
@@
     (add_net "Net-(J1-Pad2)")
     (add_net "Net-(J2-Pad2)")
+  )
+  (module IHE2:Relay (layer F.Cu)
+    (at 140.35 107.65 90)
+    (fp_text reference K2 (at 13 0 180) (layer F.SilkS)
+      (effects (font (size 1 1) (thickness 0.15)))
+    )
+    (fp_text value RELAY (at -6.01 0.67 90) (layer F.SilkS) hide
+      (effects (font (size 1 1) (thickness 0.15)))
+    )
+    (fp_line (start 11.778 -2.5) (end -9.4 -2.5) (layer F.SilkS) (width 0.15))
+    (fp_line (start 11.778 2.5) (end 11.778 -2.5) (layer F.SilkS) (width 0.15))
+    (fp_line (start -9.4 2.5) (end 11.778 2.5) (layer F.SilkS) (width 0.15))
+    (fp_line (start -9.4 -2.5) (end -9.4 2.5) (layer F.SilkS) (width 0.15))
+    (pad 2 thru_hole circle (at -5.54 -1.45 90) (size 1.778 1.778) (drill 1) (layers *.Cu *.Mask F.SilkS)
+      (net 4 "Net-(D3-Pad1)"))
+    (pad 1 thru_hole circle (at -8.08 -1.45 90) (size 1.778 1.778) (drill 1) (layers *.Cu *.Mask F.SilkS)
+      (net 3 +5V))
+    (pad 3 thru_hole circle (at 2.06 -1.45 90) (size 1.778 1.778) (drill 1.2) (layers *.Cu *.Mask F.SilkS)
+      (net 15 "Net-(F2-Pad1)"))
+    (pad 4 thru_hole circle (at 9.68 -1.45 90) (size 1.778 1.778) (drill 1.2) (layers *.Cu *.Mask F.SilkS)
+      (net 7 "Net-(J2-Pad2)"))
+  )
+  (module IHE:Relay (layer F.Cu)
+    (at 122.35 107.65 90)
+    (fp_text reference K1 (at 13 0 180) (layer F.SilkS)
+      (effects (font (size 1 1) (thickness 0.15)))
+    )
+    (fp_text value RELAY (at -6.01 0.67 90) (layer F.SilkS) hide
+      (effects (font (size 1 1) (thickness 0.15)))
+    )
+    (fp_line (start -9.4 -2.5) (end -9.4 2.5) (layer F.SilkS) (width 0.15))
+    (fp_line (start -9.4 2.5) (end 11.778 2.5) (layer F.SilkS) (width 0.15))
+    (fp_line (start 11.778 2.5) (end 11.778 -2.5) (layer F.SilkS) (width 0.15))
+    (fp_line (start 11.778 -2.5) (end -9.4 -2.5) (layer F.SilkS) (width 0.15))
+    (pad 4 thru_hole circle (at 9.68 -1.45 90) (size 1.778 1.778) (drill 1.2) (layers *.Cu *.Mask F.SilkS)
+      (net 6 "Net-(J1-Pad2)"))
+    (pad 3 thru_hole circle (at 2.06 -1.45 90) (size 1.778 1.778) (drill 1.2) (layers *.Cu *.Mask F.SilkS)
+      (net 13 "Net-(F1-Pad1)"))
+    (pad 1 thru_hole circle (at -8.08 -1.45 90) (size 1.778 1.778) (drill 1) (layers *.Cu *.Mask F.SilkS)
+      (net 3 +5V))
+    (pad 2 thru_hole circle (at -5.54 -1.45 90) (size 1.778 1.778) (drill 1) (layers *.Cu *.Mask F.SilkS)
+      (net 1 "Net-(D1-Pad1)"))
   )
   (module Mounting_Holes:MountingHole_2.7mm_M2.5_Pad (layer F.Cu)
@@
     )
   )
-  (module IHE:Relay (layer F.Cu)
-    (at 122.35 107.65 90)
-    (fp_text reference K1 (at 13 0 180) (layer F.SilkS)
-      (effects (font (size 1 1) (thickness 0.15)))
-    )
-    (fp_text value RELAY (at -6.01 0.67 90) (layer F.SilkS) hide
-      (effects (font (size 1 1) (thickness 0.15)))
-    )
-    (fp_line (start -10 -2.5) (end -10 2.5) (layer F.SilkS) (width 0.15))
-    (fp_line (start -10 2.5) (end 11.778 2.5) (layer F.SilkS) (width 0.15))
-    (fp_line (start 11.778 2.5) (end 11.778 -2.5) (layer F.SilkS) (width 0.15))
-    (fp_line (start 11.778 -2.5) (end -10 -2.5) (layer F.SilkS) (width 0.15))
-    (pad 4 thru_hole circle (at 10.16 -1.45 90) (size 1.778 1.778) (drill 0.762) (layers *.Cu *.Mask F.SilkS)
-      (net 6 "Net-(J1-Pad2)"))
-    (pad 3 thru_hole circle (at 2.06 -1.45 90) (size 1.778 1.778) (drill 0.762) (layers *.Cu *.Mask F.SilkS)
-      (net 13 "Net-(F1-Pad1)"))
-    (pad 1 thru_hole circle (at -8.08 -1.45 90) (size 1.778 1.778) (drill 0.762) (layers *.Cu *.Mask F.SilkS)
-      (net 3 +5V))
-    (pad 2 thru_hole circle (at -5.54 -1.45 90) (size 1.778 1.778) (drill 0.762) (layers *.Cu *.Mask F.SilkS)
-      (net 1 "Net-(D1-Pad1)"))
-  )
   (module TO_SOT_Packages_THT:TO-92_Inline_Narrow_Oval (layer F.Cu)
     (at 127.35 108.65)
@@
       (net 1 "Net-(D1-Pad1)"))
     (model ${KISYS3DMOD}/TO_SOT_Packages_THT.3dshapes/TO-92_Inline_Narrow_Oval.wrl
-      (at (xyz 0.05 0 0))
+      (offset (xyz 1.269999980926514 0 0))
       (scale (xyz 1 1 1))
       (rotate (xyz 0 0 -90))
@@
       (net 4 "Net-(D3-Pad1)"))
     (model ${KISYS3DMOD}/TO_SOT_Packages_THT.3dshapes/TO-92_Inline_Narrow_Oval.wrl
-      (at (xyz 0.05 0 0))
+      (offset (xyz 1.269999980926514 0 0))
       (scale (xyz 1 1 1))
       (rotate (xyz 0 0 -90))
@@
     (tags "resistor 0805")
     (attr smd)
-    (fp_text reference R1 (at 0 -2 360) (layer F.SilkS)
+    (fp_text reference R1 (at 0 -2) (layer F.SilkS)
       (effects (font (size 1 1) (thickness 0.15)))
     )
@@
     (tags "resistor 0805")
     (attr smd)
-    (fp_text reference R2 (at 0 -2 360) (layer F.SilkS)
+    (fp_text reference R2 (at 0 -2) (layer F.SilkS)
       (effects (font (size 1 1) (thickness 0.15)))
     )
@@
     (tags "resistor 0805")
     (attr smd)
-    (fp_text reference R5 (at 3.5 1 360) (layer F.SilkS)
+    (fp_text reference R5 (at 3.5 1) (layer F.SilkS)
       (effects (font (size 1 1) (thickness 0.15)))
     )
@@
     (tags "resistor 0805")
     (attr smd)
-    (fp_text reference R6 (at 0 -2 360) (layer F.SilkS)
+    (fp_text reference R6 (at 0 -2) (layer F.SilkS)
       (effects (font (size 1 1) (thickness 0.15)))
     )
@@
       (net 16 "Net-(F2-Pad2)"))
   )
-  (module IHE:Relay (layer F.Cu)
-    (at 140.35 107.65 90)
-    (fp_text reference K2 (at 13 0 180) (layer F.SilkS)
-      (effects (font (size 1 1) (thickness 0.15)))
-    )
-    (fp_text value RELAY (at -6.01 0.67 90) (layer F.SilkS) hide
-      (effects (font (size 1 1) (thickness 0.15)))
-    )
-    (fp_line (start -10 -2.5) (end -10 2.5) (layer F.SilkS) (width 0.15))
-    (fp_line (start -10 2.5) (end 11.778 2.5) (layer F.SilkS) (width 0.15))
-    (fp_line (start 11.778 2.5) (end 11.778 -2.5) (layer F.SilkS) (width 0.15))
-    (fp_line (start 11.778 -2.5) (end -10 -2.5) (layer F.SilkS) (width 0.15))
-    (pad 4 thru_hole circle (at 10.16 -1.45 90) (size 1.778 1.778) (drill 0.762) (layers *.Cu *.Mask F.SilkS)
-      (net 7 "Net-(J2-Pad2)"))
-    (pad 3 thru_hole circle (at 2.06 -1.45 90) (size 1.778 1.778) (drill 0.762) (layers *.Cu *.Mask F.SilkS)
-      (net 15 "Net-(F2-Pad1)"))
-    (pad 1 thru_hole circle (at -8.08 -1.45 90) (size 1.778 1.778) (drill 0.762) (layers *.Cu *.Mask F.SilkS)
-      (net 3 +5V))
-    (pad 2 thru_hole circle (at -5.54 -1.45 90) (size 1.778 1.778) (drill 0.762) (layers *.Cu *.Mask F.SilkS)
-      (net 4 "Net-(D3-Pad1)"))
-  )
   (module Pin_Headers:Pin_Header_Straight_2x02_Pitch2.54mm (layer F.Cu)
     (at 131.05 123.95 90)
@@
     (fp_circle (center 0 0) (end 2.95 0) (layer F.CrtYd) (width 0.05))
     (pad 1 thru_hole circle (at 0 0) (size 5.4 5.4) (drill 2.7) (layers *.Cu *.Mask))
+  )
+  (gr_text "Rev B" (at 117.35 92.15 270) (layer F.SilkS)
+    (effects (font (size 1.5 1.5) (thickness 0.3)))
   )
   (gr_line (start 158.35 128.15) (end 158.35 80.15) (angle 90) (layer Edge.Cuts) (width 0.15))
@@
   (segment (start 145.35 123) (end 142.24 123) (width 0.25) (layer F.Cu) (net 5))
   (segment (start 142.24 123) (end 140.89 121.65) (width 0.25) (layer F.Cu) (net 5))
-  (segment (start 120.9 97.49) (end 120.9 89.1) (width 2) (layer F.Cu) (net 6))
   (segment (start 120.9 89.1) (end 123.35 86.65) (width 2) (layer F.Cu) (net 6))
-  (segment (start 138.9 97.49) (end 138.9 89.1) (width 2) (layer F.Cu) (net 7))
+  (segment (start 120.9 96.15) (end 120.9 97.97) (width 2) (layer F.Cu) (net 6))
+  (segment (start 120.9 97.49) (end 120.9 96.15) (width 2) (layer F.Cu) (net 6))
+  (segment (start 120.9 96.15) (end 120.9 89.1) (width 2) (layer F.Cu) (net 6))
   (segment (start 138.9 89.1) (end 141.35 86.65) (width 2) (layer F.Cu) (net 7))
+  (segment (start 138.9 96.15) (end 138.9 97.97) (width 2) (layer F.Cu) (net 7))
+  (segment (start 138.9 97.49) (end 138.9 96.15) (width 2) (layer F.Cu) (net 7))
+  (segment (start 138.9 96.15) (end 138.9 89.1) (width 2) (layer F.Cu) (net 7))
   (segment (start 131.05 121.41) (end 131.35 121) (width 0.25) (layer F.Cu) (net 8) (status 10))
   (segment (start 131.35 121) (end 127.35 117) (width 0.25) (layer F.Cu) (net 8))

Commit message: use official footprint libs
Parts:
- K1: footprint IHE:Relay -> Relay_THT:Relay_SPST_TE_PCN-1xxD3MHZ
- K2: footprint IHE2:Relay -> Relay_THT:Relay_SPST_TE_PCN-1xxD3MHZ
- R1, R2: value 10kΩ -> 240Ω
- moved K1 8.21 mm to (120.9, 115.7)
- moved K2 8.21 mm to (138.9, 115.7)
